Commit message: Small fixes.

File: toad_description/urdf/hokuyo_utm30lx.urdf.xacro (robot description, xacro)
@@ -24,5 +24,4 @@
       <geometry>
       <box size="0.058 0.058 0.087" />
-      <!--<mesh filename="package://hector_sensors_description/meshes/hokuyo_utm30lx/hokuyo_utm_30lx.stl"/>-->
     </geometry>
     </collision>

File: toad_description/urdf/toad.urdf.xacro (robot description, xacro)
@@ -6,5 +6,4 @@
 name="toad">
   <include filename="$(find p2os_urdf)/defs/pioneer3at_body.xacro"/>
-  <!--include filename="$(find hector_sensors_description)/urdf/hokuyo_utm30lx.urdf.xacro"/-->
   <include filename="$(find toad_description)/urdf/hokuyo_utm30lx.urdf.xacro"/>
   <xacro:p3at_front suffix="left" reflect="1"/>
