Commit message: Simulation of stereo camera.

File: toad_description/urdf/toad.urdf.xacro (robot description, xacro)
@@ -11,3 +11,179 @@
   <xacro:p3at_back suffix="right" reflect="-1"/>
   <xacro:p3at_gazebo_ext/>
+  <joint name="p3at_velodyne_joint" type="fixed">
+		<origin xyz="0 0 0.5" rpy="0 0 0"/>
+		<parent link="base_link"/>
+		<child link="velodyne_link"/>
+	</joint>
+	<joint name="p3at_left_cam_joint" type="fixed">
+		<origin xyz="0 -0.2 0.4" rpy="0 0 0"/>
+		<parent link="base_link"/>
+		<child link="left_cam_link"/>
+	</joint>
+	<joint name="p3at_right_cam_joint" type="fixed">
+		<origin xyz="0 0.2 0.4" rpy="0 0 0"/>
+		<parent link="base_link"/>
+		<child link="right_cam_link"/>
+	</joint>
+	<link name="velodyne_link">
+		<inertial>
+			<mass value="1.0"/>
+			<origin xyz="0 0 0"/>
+			<inertia ixx="1.0" ixy="0.0" ixz="0.0"
+				 iyy="1.0" iyz="0.0" izz="1.0"/>
+  	 	</inertial>
+	<visual name="base_visual">
+		<origin xyz="0 0 0" rpy="0 0 0"/>
+		<geometry name="pioneer_geom">
+			<cylinder length="0.15" radius="0.07"/>
+		</geometry>
+		<material name="velodyneGrey">
+        <color rgba="0.6 0.6 0.6 1"/>
+    </material>
+	</visual>
+	<collision>
+		<origin xyz="0 0 0" rpy="0 0 0"/>
+		<geometry>
+			<cylinder length="0.15" radius="0.05"/>
+		</geometry>
+	</collision>
+	</link>
+	<link name="left_cam_link">
+		<inertial>
+			<mass value="0.2"/>
+			<origin xyz="0 0 0"/>
+			<inertia ixx="1.0" ixy="0.0" ixz="0.0"
+				 iyy="1.0" iyz="0.0" izz="1.0"/>
+  	 	</inertial>
+	<visual>
+		<origin xyz="0 0 0" rpy="0 0 0"/>
+		<geometry>
+			<box size="0.025 .05 .05"/>
+		</geometry>
+		<material name="cameraGray">
+        <color rgba="0.4 0.4 0.4 1"/>
+    </material>
+	</visual>
+	<collision>
+		<origin xyz="0 0 0" rpy="0 0 0"/>
+		<geometry>
+			<box size="0.025 .05 .05"/>
+		</geometry>
+	</collision>
+	</link>
+	<link name="right_cam_link">
+		<inertial>
+			<mass value="0.2"/>
+			<origin xyz="0 0 0"/>
+			<inertia ixx="1.0" ixy="0.0" ixz="0.0"
+				 iyy="1.0" iyz="0.0" izz="1.0"/>
+  	 	</inertial>
+	<visual>
+		<origin xyz="0 0 0" rpy="0 0 0"/>
+		<geometry>
+			<box size="0.025 .05 .05"/>
+		</geometry>
+		<material name="cameraGray">
+        <color rgba="0.4 0.4 0.4 1"/>
+    </material>
+	</visual>
+	<collision>
+		<origin xyz="0 0 0" rpy="0 0 0"/>
+		<geometry>
+			<box size="0.025 .05 .05"/>
+		</geometry>
+	</collision>
+	</link>
+  <gazebo reference="left_cam_link">
+    <sensor type="multicamera" name="stereo_camera">
+      <update_rate>30.0</update_rate>
+      <camera name="left">
+        <pose>0 0 0 0 0 0</pose>
+        <horizontal_fov>0.733038285</horizontal_fov>
+        <image>
+          <width>640</width>
+          <height>480</height>
+          <format>R8G8B8</format>
+        </image>
+        <clip>
+          <near>0.02</near>
+          <far>300</far>
+        </clip>
+        <noise>
+          <type>gaussian</type>
+          <mean>0.0</mean>
+          <stddev>0.007</stddev>
+        </noise>
+      </camera>
+      <camera name="right">
+        <pose>0 -0.4 0 0 0 0</pose>
+        <horizontal_fov>0.733038285</horizontal_fov>
+        <image>
+          <width>640</width>
+          <height>480</height>
+          <format>R8G8B8</format>
+        </image>
+        <clip>
+          <near>0.02</near>
+          <far>300</far>
+        </clip>
+        <noise>
+          <type>gaussian</type>
+          <mean>0.0</mean>
+          <stddev>0.007</stddev>
+        </noise>
+      </camera>
+      <plugin name="stereo_camera_controller" filename="libgazebo_ros_multicamera.so">
+        <alwaysOn>true</alwaysOn>
+        <updateRate>0.0</updateRate>
+        <cameraName>stereo</cameraName>
+        <imageTopicName>image_color</imageTopicName>
+        <cameraInfoTopicName>camera_info</cameraInfoTopicName>
+        <frameName>left_cam_link</frameName>
+        <rightFrameName>right_cam_link</rightFrameName>
+        <hackBaseline>0.0</hackBaseline>
+        <distortionK1>0.0</distortionK1>
+        <distortionK2>0.0</distortionK2>
+        <distortionK3>0.0</distortionK3>
+        <distortionT1>0.0</distortionT1>
+        <distortionT2>0.0</distortionT2>
+      </plugin>
+    </sensor>
+  </gazebo>
+ <gazebo reference="velodyne_link">
+      <sensor type="ray" name="ray_sensor">
+        <always_on>true</always_on>
+        <update_rate>10.0</update_rate>
+        <pose>0 0 0 0 0 0</pose>
+        <visualize>false</visualize>
+        <ray>
+          <scan>
+            <horizontal>
+              <samples>21875</samples>
+              <resolution>1.0</resolution>
+              <min_angle>-3.14</min_angle>
+              <max_angle>3.14</max_angle>
+            </horizontal>
+            <!--vertical>
+              <samples>32</samples>
+              <resolution>1.0</resolution>
+              <min_angle>-0.535</min_angle>
+              <max_angle>0.186132</max_angle>
+            </vertical-->
+          </scan>
+          <range>
+            <min>1.0</min>
+            <max>20.0</max>
+            <resolution>0.01</resolution>
+          </range>
+        </ray>
+        <plugin name="gazebo_ros_ray_sensor_controller" filename="libgazebo_ros_block_laser.so">
+          <gaussianNoise>0.005</gaussianNoise>
+          <alwaysOn>true</alwaysOn>
+          <updateRate>10.0</updateRate>
+          <topicName>velodyne_cloud</topicName>
+          <frameName>velodyne_link</frameName>
+        </plugin>
+      </sensor>
+    </gazebo>
 </robot>

Commit message: Added robot_pose_ekf.

File: toad_description/urdf/toad.urdf.xacro (robot description, xacro)
@@ -16,4 +16,9 @@
 		<child link="velodyne_link"/>
 	</joint>
+	<joint name="p3at_imu_joint" type="fixed">
+		<origin xyz="0 -0.2 0.5" rpy="0 0 0"/>
+		<parent link="base_link"/>
+		<child link="imu_link"/>
+	</joint>
 	<joint name="p3at_left_cam_joint" type="fixed">
 		<origin xyz="0 -0.2 0.4" rpy="0 0 0"/>
@@ -49,4 +54,27 @@
 	</collision>
 	</link>
+	<link name="imu_link">
+		<inertial>
+			<mass value="0.1"/>
+			<origin xyz="0 0 0"/>
+			<inertia ixx="1.0" ixy="0.0" ixz="0.0"
+				 iyy="1.0" iyz="0.0" izz="1.0"/>
+  	 	</inertial>
+	<visual name="imu_vis">
+		<origin xyz="0 0 0" rpy="0 0 0"/>
+		<geometry>
+			<box size="0.01 .01 .01"/>
+		</geometry>
+		<material name="imuBlack">
+        <color rgba="0.9 0.9 0.9 1"/>
+    </material>
+	</visual>
+	<collision>
+		<origin xyz="0 0 0" rpy="0 0 0"/>
+		<geometry>
+			<box size="0.01 .01 .01"/>
+		</geometry>
+	</collision>
+	</link>
 	<link name="left_cam_link">
 		<inertial>
@@ -56,5 +84,5 @@
 				 iyy="1.0" iyz="0.0" izz="1.0"/>
   	 	</inertial>
-	<visual>
+	<visual name="lcvis">
 		<origin xyz="0 0 0" rpy="0 0 0"/>
 		<geometry>
@@ -79,5 +107,5 @@
 				 iyy="1.0" iyz="0.0" izz="1.0"/>
   	 	</inertial>
-	<visual>
+	<visual name="rcvis">
 		<origin xyz="0 0 0" rpy="0 0 0"/>
 		<geometry>
@@ -95,4 +123,29 @@
 	</collision>
 	</link>
+	<gazebo>
+	<plugin name="imu_sim" filename="libhector_gazebo_ros_imu.so">
+      <updateRate>20.0</updateRate>
+      <bodyName>imu_link</bodyName>
+      <topicName>/imu_3dm_node/imu/data</topicName>
+      <rpyOffsets>0 0 0</rpyOffsets> <!-- deprecated -->
+      <gaussianNoise>0</gaussianNoise>  <!-- deprecated -->
+      <accelDrift>0.5 0.5 0.5</accelDrift>
+      <accelGaussianNoise>0.35 0.35 0.3</accelGaussianNoise>
+      <rateDrift>0.1 0.1 0.1</rateDrift>
+      <rateGaussianNoise>0.05 0.05 0.015</rateGaussianNoise>
+      <headingDrift>0.1</headingDrift>
+      <headingGaussianNoise>0.05</headingGaussianNoise>
+    </plugin>
+    <plugin name="gps_sim" filename="libhector_gazebo_ros_gps.so">
+      <updateRate>10.0</updateRate>
+      <bodyName>imu_link</bodyName>
+      <topicName>/imu_3dm_node/nav/fix</topicName>
+      <velocityTopicName>/imu_3dm_node/nav/fix_velocity</velocityTopicName>
+      <drift>5.0 5.0 5.0</drift>
+      <gaussianNoise>0.01 0.01 0.01</gaussianNoise>
+      <velocityDrift>0 0 0</velocityDrift>
+      <velocityGaussianNoise>0.05 0.05 0.05</velocityGaussianNoise>
+    </plugin>
+	</gazebo>
   <gazebo reference="left_cam_link">
     <sensor type="multicamera" name="stereo_camera">

Commit message: URDF updates (stereo/navigation related).

File: toad_description/urdf/toad.urdf.xacro (robot description, xacro)
@@ -34,5 +34,5 @@
 		<inertial>
 			<mass value="1.0"/>
-			<origin xyz="0 0 0"/>
+			<origin xyz="0 0 0" rpy="0 0 0"/>
 			<inertia ixx="1.0" ixy="0.0" ixz="0.0"
 				 iyy="1.0" iyz="0.0" izz="1.0"/>
@@ -57,5 +57,5 @@
 		<inertial>
 			<mass value="0.1"/>
-			<origin xyz="0 0 0"/>
+			<origin xyz="0 0 0" rpy="0 0 0"/>
 			<inertia ixx="1.0" ixy="0.0" ixz="0.0"
 				 iyy="1.0" iyz="0.0" izz="1.0"/>
@@ -80,5 +80,5 @@
 		<inertial>
 			<mass value="0.2"/>
-			<origin xyz="0 0 0"/>
+			<origin xyz="0 0 0" rpy="0 0 0"/>
 			<inertia ixx="1.0" ixy="0.0" ixz="0.0"
 				 iyy="1.0" iyz="0.0" izz="1.0"/>
@@ -103,5 +103,5 @@
 		<inertial>
 			<mass value="0.2"/>
-			<origin xyz="0 0 0"/>
+			<origin xyz="0 0 0" rpy="0 0 0"/>
 			<inertia ixx="1.0" ixy="0.0" ixz="0.0"
 				 iyy="1.0" iyz="0.0" izz="1.0"/>
@@ -123,4 +123,16 @@
 	</collision>
 	</link>
+	<joint name="p3at_left_cam_optical_joint" type="fixed">
+		<origin xyz="0 0 0" rpy="1.57 3.14 1.57"/>
+		<parent link="left_cam_link"/>
+		<child link="left_cam_optical_link"/>
+	</joint>
+	<joint name="p3at_right_cam_optical_joint" type="fixed">
+		<origin xyz="0 0 0" rpy="1.57 3.14 1.57"/>
+		<parent link="right_cam_link"/>
+		<child link="right_cam_optical_link"/>
+	</joint>
+	<link name="left_cam_optical_link"/>
+	<link name="right_cam_optical_link"/>
 	<gazebo>
 	<plugin name="imu_sim" filename="libhector_gazebo_ros_imu.so">
@@ -146,4 +158,6 @@
       <velocityDrift>0 0 0</velocityDrift>
       <velocityGaussianNoise>0.05 0.05 0.05</velocityGaussianNoise>
+      <referenceLatitude>49.207387</referenceLatitude>
+      <referenceLongitude>16.609840</referenceLongitude>
     </plugin>
 	</gazebo>
@@ -193,6 +207,6 @@
         <imageTopicName>image_raw</imageTopicName>
         <cameraInfoTopicName>camera_info</cameraInfoTopicName>
-        <frameName>left_cam_link</frameName>
-        <rightFrameName>right_cam_link</rightFrameName>
+        <frameName>left_cam_optical_link</frameName>
+        <rightFrameName>right_cam_optical_link</rightFrameName>
         <hackBaseline>0.4</hackBaseline>
         <distortionK1>0.0</distortionK1>

Commit message: Added Hokuyo laser range finder.

File: toad_description/urdf/toad.urdf.xacro (robot description, xacro)
@@ -6,4 +6,6 @@
 name="toad">
   <include filename="$(find p2os_urdf)/defs/pioneer3at_body.xacro"/>
+  <!--include filename="$(find hector_sensors_description)/urdf/hokuyo_utm30lx.urdf.xacro"/-->
+  <include filename="$(find toad_description)/urdf/hokuyo_utm30lx.urdf.xacro"/>
   <xacro:p3at_front suffix="left" reflect="1"/>
   <xacro:p3at_front suffix="right" reflect="-1"/>
@@ -135,4 +137,8 @@
 	<link name="left_cam_optical_link"/>
 	<link name="right_cam_optical_link"/>
+	<!-- Hokuyo UTM-30LX mounted upside down -->
+	<xacro:hokuyo_utm30lx name="hokuyo" parent="base_link" ros_topic="/scan" update_rate="10" ray_count="1080" min_angle="-135" max_angle="135">
+  	<origin xyz="0.32 0.0 0.2" rpy="${M_PI} 0 0"/>
+	</xacro:hokuyo_utm30lx>
 	<gazebo>
 	<plugin name="imu_sim" filename="libhector_gazebo_ros_imu.so">
@@ -164,5 +170,5 @@
   <gazebo reference="left_cam_link">
     <sensor type="multicamera" name="stereo_camera">
-      <update_rate>15.0</update_rate>
+      <update_rate>5.0</update_rate>
       <camera name="left">
         <pose>0 0 0 0 0 0</pose>
@@ -219,5 +225,5 @@
   </gazebo>
  <gazebo reference="velodyne_link">
-    <sensor type="gpu_ray" name="head_hokuyo_sensor">
+    <sensor type="gpu_ray" name="velodyne">
       <pose>0 0 0 0 0 0</pose>
       <visualize>false</visualize>
@@ -234,5 +240,5 @@
         <range>
           <min>0.3</min>
-          <max>10.0</max>
+          <max>5.0</max>
           <resolution>0.01</resolution>
         </range>

Commit message: URDF tuning.

File: toad_description/urdf/toad.urdf.xacro (robot description, xacro)
@@ -24,10 +24,10 @@
 	</joint>
 	<joint name="p3at_left_cam_joint" type="fixed">
+		<origin xyz="0 0.2 0.4" rpy="0 0 0"/>
+		<parent link="base_link"/>
+		<child link="left_cam_link"/>
+	</joint>
+	<joint name="p3at_right_cam_joint" type="fixed">
 		<origin xyz="0 -0.2 0.4" rpy="0 0 0"/>
-		<parent link="base_link"/>
-		<child link="left_cam_link"/>
-	</joint>
-	<joint name="p3at_right_cam_joint" type="fixed">
-		<origin xyz="0 0.2 0.4" rpy="0 0 0"/>
 		<parent link="base_link"/>
 		<child link="right_cam_link"/>

Commit message: Changes to Gazebo world file - textures now don't flickr and simulation is faster.

File: toad_description/urdf/toad.urdf.xacro (robot description, xacro)
@@ -14,20 +14,20 @@
   <xacro:p3at_gazebo_ext/>
   <joint name="p3at_velodyne_joint" type="fixed">
-		<origin xyz="0 0 0.5" rpy="0 0 0"/>
+		<origin xyz="0.05 0 0.8" rpy="0 0 0"/>
 		<parent link="base_link"/>
 		<child link="velodyne_link"/>
 	</joint>
 	<joint name="p3at_imu_joint" type="fixed">
-		<origin xyz="0 -0.2 0.5" rpy="0 0 0"/>
+		<origin xyz="0.05 0.2 0.72" rpy="0 0 0"/>
 		<parent link="base_link"/>
 		<child link="imu_link"/>
 	</joint>
 	<joint name="p3at_left_cam_joint" type="fixed">
-		<origin xyz="0 0.2 0.4" rpy="0 0 0"/>
+		<origin xyz="0.1 0.2 0.67" rpy="0 ${20 * M_PI/180} 0"/>
 		<parent link="base_link"/>
 		<child link="left_cam_link"/>
 	</joint>
 	<joint name="p3at_right_cam_joint" type="fixed">
-		<origin xyz="0 -0.2 0.4" rpy="0 0 0"/>
+		<origin xyz="0.1 -0.2 0.67" rpy="0 ${20 * M_PI/180} 0"/>
 		<parent link="base_link"/>
 		<child link="right_cam_link"/>

Commit message: Some changes for velodyne.

File: toad_description/urdf/toad.urdf.xacro (robot description, xacro)
@@ -13,7 +13,7 @@
   <xacro:p3at_gazebo_ext/>
   <joint name="p3at_velodyne_joint" type="fixed">
-		<origin xyz="0.05 0 0.8" rpy="0 0 0"/>
-		<parent link="base_link"/>
-		<child link="velodyne_link"/>
+		<origin xyz="0.05 0 0.8" rpy="0 0 ${-90 * M_PI/180}"/>
+		<parent link="base_link"/>
+		<child link="velodyne"/>
 	</joint>
 	<joint name="p3at_imu_joint" type="fixed">
@@ -23,14 +23,14 @@
 	</joint>
 	<joint name="p3at_left_cam_joint" type="fixed">
-		<origin xyz="0.1 0.2 0.67" rpy="0 ${20 * M_PI/180} 0"/>
+		<origin xyz="0.1 0.2 0.67" rpy="0 ${16 * M_PI/180} 0"/>
 		<parent link="base_link"/>
 		<child link="left_cam_link"/>
 	</joint>
 	<joint name="p3at_right_cam_joint" type="fixed">
-		<origin xyz="0.1 -0.2 0.67" rpy="0 ${20 * M_PI/180} 0"/>
+		<origin xyz="0.1 -0.2 0.67" rpy="0 ${16 * M_PI/180} 0"/>
 		<parent link="base_link"/>
 		<child link="right_cam_link"/>
 	</joint>
-	<link name="velodyne_link">
+	<link name="velodyne">
 		<inertial>
 			<mass value="1.0"/>
@@ -223,5 +223,5 @@
     </sensor>
   </gazebo>
- <gazebo reference="velodyne_link">
+ <gazebo reference="velodyne">
     <sensor type="gpu_ray" name="velodyne">
       <pose>0 0 0 0 0 0</pose>
@@ -250,5 +250,5 @@
       <plugin name="gazebo_ros_velodyne_laser_controller" filename="libgazebo_ros_gpu_laser.so">
         <topicName>/velodyne/scan</topicName>
-        <frameName>velodyne_link</frameName>
+        <frameName>velodyne</frameName>
       </plugin>
     </sensor>

Commit message: Recent changes.

File: toad_description/urdf/toad.urdf.xacro (robot description, xacro)
@@ -23,5 +23,6 @@
 	</joint>
 	<joint name="p3at_left_cam_joint" type="fixed">
-		<origin xyz="0.1 0.2 0.67" rpy="0 ${16 * M_PI/180} 0"/>
+		<!--origin xyz="0.1 0.2 0.67" rpy="0 ${16 * M_PI/180} 0"/-->
+		<origin xyz="0.093 0.266 0.669" rpy="-0.0064 0.2913862 -0.00165"/>
 		<parent link="base_link"/>
 		<child link="left_cam_link"/>

Commit message: Update to include Hokuyo.

File: toad_description/urdf/toad.urdf.xacro (robot description, xacro)
@@ -5,6 +5,6 @@
        xmlns:xacro="http://ros.org/wiki/xacro"
 name="toad">
-  <include filename="$(find p2os_urdf)/defs/pioneer3at_body.xacro"/>
-  <include filename="$(find toad_description)/urdf/hokuyo_utm30lx.urdf.xacro"/>
+  <xacro:include filename="$(find p2os_urdf)/defs/pioneer3at_body.xacro"/>
+  <xacro:include filename="$(find toad_description)/urdf/hokuyo_utm30lx.urdf.xacro"/>
   <xacro:p3at_front suffix="left" reflect="1"/>
   <xacro:p3at_front suffix="right" reflect="-1"/>
@@ -13,5 +13,5 @@
   <xacro:p3at_gazebo_ext/>
   <joint name="p3at_velodyne_joint" type="fixed">
-		<origin xyz="0.05 0 0.8" rpy="0 0 ${-90 * M_PI/180}"/>
+		<origin xyz="0 0 0.8" rpy="0 0 ${-90 * M_PI/180}"/>
 		<parent link="base_link"/>
 		<child link="velodyne"/>
@@ -139,5 +139,5 @@
 	<!-- Hokuyo UTM-30LX mounted upside down -->
 	<xacro:hokuyo_utm30lx name="hokuyo" parent="base_link" ros_topic="/scan" update_rate="10" ray_count="1080" min_angle="-135" max_angle="135">
-  	<origin xyz="0.32 0.0 0.2" rpy="${M_PI} 0 0"/>
+  	<origin xyz="0.25 0.0 0.35" rpy="0 0 0"/>
 	</xacro:hokuyo_utm30lx>
 	<gazebo>
